File: motor_driver_module.sch (EAGLE design)
At the start: 48 parts, among them IC3 LTC6087, IC4 LTC6087, IC7 DRV8833RTY, IC8 DRV8833RTY, P1 BAT+, P10 MD2, P11 MA_IN1, P12 MA_IN2, P13 MB_IN1, P14 MB_IN2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

Commit message: More rerouting. Minimal size does not look promising as of right now.
Connections:
- net MOTOR_A_BEMF: now also R3A.1; no longer R3A.2
- net MOTOR_A_OUT1: now also R33B.2; no longer R33A.1
- net MOTOR_A_OUT2: now also R33A.2; no longer R33B.1
- net MOTOR_B_BEMF: now also R3B.1; no longer R3B.2
- net MOTOR_C_BEMF: now also R3C.1; no longer R3C.2
- net MOTOR_D_BEMF: now also R3D.1; no longer R3D.2
- net N$30: now also R33B.1; no longer R33A.2
- net N$31: now also R33A.1; no longer R33B.2
- net N$34: now also R3D.2; no longer R3D.1
- net N$35: now also R3C.2; no longer R3C.1
- net N$36: now also R3A.2; no longer R3A.1
- net N$37: now also R3B.2; no longer R3B.1
Other:
- moved on the sheet: R33A, R33B, R3A, R3B, R3C, R3D
Changed lines of the file:
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@@
 <instance part="GND33" gate="1" x="180.34" y="45.72"/>
 <instance part="GND46" gate="1" x="180.34" y="119.38"/>
-<instance part="R33" gate="A" x="140.97" y="170.18" smashed="yes">
-<attribute name="NAME" x="138.938" y="167.64" size="1.27" layer="95" ratio="10"/>
-<attribute name="VALUE" x="139.7" y="171.196" size="1.27" layer="96" ratio="10"/>
-</instance>
-<instance part="R33" gate="B" x="140.97" y="165.1" smashed="yes">
-<attribute name="NAME" x="139.192" y="162.56" size="1.27" layer="95" ratio="10"/>
-<attribute name="VALUE" x="139.7" y="165.862" size="1.27" layer="96" ratio="10"/>
-</instance>
 <instance part="R33" gate="C" x="140.97" y="129.54" smashed="yes">
 <attribute name="NAME" x="138.684" y="127.254" size="1.27" layer="95" ratio="10"/>
@@
 <instance part="GND24" gate="1" x="111.76" y="7.62"/>
 <instance part="R8" gate="C" x="147.32" y="158.75" rot="R90"/>
-<instance part="R3" gate="A" x="171.45" y="167.64" smashed="yes">
-<attribute name="NAME" x="169.672" y="165.354" size="1.27" layer="95" ratio="10"/>
-<attribute name="VALUE" x="169.926" y="168.656" size="1.27" layer="96" ratio="10"/>
-</instance>
-<instance part="R3" gate="B" x="171.45" y="132.08"/>
-<instance part="R3" gate="C" x="171.45" y="93.98"/>
-<instance part="R3" gate="D" x="171.45" y="58.42"/>
+<instance part="R3" gate="A" x="171.45" y="167.64" smashed="yes" rot="R180">
+<attribute name="NAME" x="173.228" y="169.926" size="1.27" layer="95" ratio="10" rot="R180"/>
+<attribute name="VALUE" x="172.974" y="166.624" size="1.27" layer="96" ratio="10" rot="R180"/>
+</instance>
+<instance part="R3" gate="B" x="171.45" y="132.08" rot="R180"/>
+<instance part="R3" gate="C" x="171.45" y="93.98" rot="R180"/>
+<instance part="R3" gate="D" x="171.45" y="58.42" rot="R180"/>
 <instance part="P3" gate="1" x="304.8" y="160.02" smashed="yes">
 <attribute name="NAME" x="289.56" y="160.02" size="1.778" layer="95"/>
@@
 <instance part="R1" gate="C" x="147.32" y="85.09" rot="R90"/>
 <instance part="R1" gate="B" x="147.32" y="49.53" rot="R90"/>
+<instance part="R33" gate="B" x="140.97" y="170.18" rot="R180"/>
+<instance part="R33" gate="A" x="140.97" y="165.1" rot="R180"/>
 </instances>
 <busses>
@@
 <wire x1="137.16" y1="165.1" x2="132.08" y2="165.1" width="0.1524" layer="91"/>
 <label x="111.76" y="165.1" size="1.778" layer="95"/>
-<pinref part="R33" gate="B" pin="1"/>
+<pinref part="R33" gate="A" pin="2"/>
 </segment>
 <segment>
@@
 <wire x1="137.16" y1="170.18" x2="132.08" y2="170.18" width="0.1524" layer="91"/>
 <label x="111.76" y="170.18" size="1.778" layer="95"/>
-<pinref part="R33" gate="A" pin="1"/>
+<pinref part="R33" gate="B" pin="2"/>
 </segment>
 <segment>
@@
 <wire x1="149.86" y1="170.18" x2="147.32" y2="170.18" width="0.1524" layer="91"/>
 <junction x="147.32" y="170.18"/>
-<pinref part="R33" gate="A" pin="2"/>
 <pinref part="IC3" gate="A" pin="+IN"/>
 <pinref part="R8" gate="D" pin="1"/>
+<pinref part="R33" gate="B" pin="1"/>
 </segment>
 </net>
@@
 <wire x1="149.86" y1="165.1" x2="147.32" y2="165.1" width="0.1524" layer="91"/>
 <junction x="147.32" y="165.1"/>
-<pinref part="R33" gate="B" pin="2"/>
 <pinref part="IC3" gate="A" pin="-IN"/>
 <pinref part="R8" gate="C" pin="2"/>
+<pinref part="R33" gate="A" pin="1"/>
 </segment>
 </net>
@@
 <segment>
 <label x="187.96" y="58.42" size="1.778" layer="95"/>
-<wire x1="175.26" y1="58.42" x2="180.34" y2="58.42" width="0.1524" layer="91"/>
 <pinref part="C44" gate="G$1" pin="1"/>
 <wire x1="180.34" y1="58.42" x2="185.42" y2="58.42" width="0.1524" layer="91"/>
 <wire x1="180.34" y1="55.88" x2="180.34" y2="58.42" width="0.1524" layer="91"/>
+<pinref part="R3" gate="D" pin="1"/>
+<wire x1="175.26" y1="58.42" x2="180.34" y2="58.42" width="0.1524" layer="91"/>
 <junction x="180.34" y="58.42"/>
-<pinref part="R3" gate="D" pin="2"/>
 </segment>
 <segment>
@@
 <segment>
 <wire x1="162.56" y1="58.42" x2="165.1" y2="58.42" width="0.1524" layer="91"/>
-<wire x1="165.1" y1="58.42" x2="167.64" y2="58.42" width="0.1524" layer="91"/>
 <wire x1="158.75" y1="68.58" x2="165.1" y2="68.58" width="0.1524" layer="91"/>
 <wire x1="165.1" y1="68.58" x2="165.1" y2="58.42" width="0.1524" layer="91"/>
+<pinref part="IC4" gate="B" pin="OUT"/>
+<pinref part="R1" gate="A" pin="2"/>
+<pinref part="R3" gate="D" pin="2"/>
+<wire x1="165.1" y1="58.42" x2="167.64" y2="58.42" width="0.1524" layer="91"/>
 <junction x="165.1" y="58.42"/>
-<pinref part="IC4" gate="B" pin="OUT"/>
-<pinref part="R3" gate="D" pin="1"/>
-<pinref part="R1" gate="A" pin="2"/>
 </segment>
 </net>
@@
 <wire x1="158.75" y1="104.14" x2="165.1" y2="104.14" width="0.1524" layer="91"/>
 <wire x1="165.1" y1="104.14" x2="165.1" y2="93.98" width="0.1524" layer="91"/>
+<pinref part="IC4" gate="A" pin="OUT"/>
+<pinref part="R1" gate="D" pin="2"/>
+<pinref part="R3" gate="C" pin="2"/>
 <wire x1="165.1" y1="93.98" x2="167.64" y2="93.98" width="0.1524" layer="91"/>
 <junction x="165.1" y="93.98"/>
-<pinref part="IC4" gate="A" pin="OUT"/>
-<pinref part="R3" gate="C" pin="1"/>
-<pinref part="R1" gate="D" pin="2"/>
 </segment>
 </net>
@@
 <wire x1="180.34" y1="93.98" x2="185.42" y2="93.98" width="0.1524" layer="91"/>
 <wire x1="180.34" y1="91.44" x2="180.34" y2="93.98" width="0.1524" layer="91"/>
+<label x="187.96" y="93.98" size="1.778" layer="95"/>
+<pinref part="R3" gate="C" pin="1"/>
 <wire x1="175.26" y1="93.98" x2="180.34" y2="93.98" width="0.1524" layer="91"/>
 <junction x="180.34" y="93.98"/>
-<label x="187.96" y="93.98" size="1.778" layer="95"/>
-<pinref part="R3" gate="C" pin="2"/>
 </segment>
 <segment>
@@
 <segment>
 <wire x1="162.56" y1="132.08" x2="165.1" y2="132.08" width="0.1524" layer="91"/>
-<wire x1="165.1" y1="132.08" x2="167.64" y2="132.08" width="0.1524" layer="91"/>
 <wire x1="158.75" y1="142.24" x2="165.1" y2="142.24" width="0.1524" layer="91"/>
 <wire x1="165.1" y1="142.24" x2="165.1" y2="132.08" width="0.1524" layer="91"/>
+<pinref part="IC3" gate="B" pin="OUT"/>
+<pinref part="R8" gate="A" pin="2"/>
+<pinref part="R3" gate="B" pin="2"/>
+<wire x1="165.1" y1="132.08" x2="167.64" y2="132.08" width="0.1524" layer="91"/>
 <junction x="165.1" y="132.08"/>
-<pinref part="IC3" gate="B" pin="OUT"/>
-<pinref part="R3" gate="B" pin="1"/>
-<pinref part="R8" gate="A" pin="2"/>
 </segment>
 </net>
 <net name="MOTOR_B_BEMF" class="0">
 <segment>
-<wire x1="175.26" y1="132.08" x2="180.34" y2="132.08" width="0.1524" layer="91"/>
 <pinref part="C42" gate="G$1" pin="1"/>
 <wire x1="180.34" y1="132.08" x2="185.42" y2="132.08" width="0.1524" layer="91"/>
 <wire x1="180.34" y1="129.54" x2="180.34" y2="132.08" width="0.1524" layer="91"/>
+<label x="187.96" y="132.08" size="1.778" layer="95"/>
+<pinref part="R3" gate="B" pin="1"/>
+<wire x1="175.26" y1="132.08" x2="180.34" y2="132.08" width="0.1524" layer="91"/>
 <junction x="180.34" y="132.08"/>
-<label x="187.96" y="132.08" size="1.778" layer="95"/>
-<pinref part="R3" gate="B" pin="2"/>
 </segment>
 <segment>
@@
 <segment>
 <wire x1="162.56" y1="167.64" x2="165.1" y2="167.64" width="0.1524" layer="91"/>
-<wire x1="165.1" y1="167.64" x2="167.64" y2="167.64" width="0.1524" layer="91"/>
 <wire x1="161.29" y1="177.8" x2="165.1" y2="177.8" width="0.1524" layer="91"/>
 <wire x1="165.1" y1="177.8" x2="165.1" y2="167.64" width="0.1524" layer="91"/>
+<pinref part="IC3" gate="A" pin="OUT"/>
+<pinref part="R8" gate="D" pin="2"/>
+<pinref part="R3" gate="A" pin="2"/>
+<wire x1="165.1" y1="167.64" x2="167.64" y2="167.64" width="0.1524" layer="91"/>
 <junction x="165.1" y="167.64"/>
-<pinref part="IC3" gate="A" pin="OUT"/>
-<pinref part="R3" gate="A" pin="1"/>
-<pinref part="R8" gate="D" pin="2"/>
 </segment>
 </net>
 <net name="MOTOR_A_BEMF" class="0">
 <segment>
-<wire x1="175.26" y1="167.64" x2="180.34" y2="167.64" width="0.1524" layer="91"/>
 <pinref part="C41" gate="G$1" pin="1"/>
 <wire x1="180.34" y1="167.64" x2="185.42" y2="167.64" width="0.1524" layer="91"/>
 <wire x1="180.34" y1="165.1" x2="180.34" y2="167.64" width="0.1524" layer="91"/>
+<label x="187.96" y="167.64" size="1.778" layer="95"/>
+<pinref part="R3" gate="A" pin="1"/>
+<wire x1="175.26" y1="167.64" x2="180.34" y2="167.64" width="0.1524" layer="91"/>
 <junction x="180.34" y="167.64"/>
-<label x="187.96" y="167.64" size="1.778" layer="95"/>
-<pinref part="R3" gate="A" pin="2"/>
-</segment>
-<segment>
+</segment>
+<segment>

Commit message: Appears more promising to use LTC6088 and discrete resistors.
Parts:
- removed C29: 0.1uF, biomimetic:CAP0402-CAP
- removed IC3, IC4: LTC6087, biomimetic:LTC6087
- removed R33, R34: 47k, OPL Eagle Library:R-4R
- added IC1: LTC6088, biomimetic:LTC6088
- added R10, R11, R12, R13, R14, R2, R4, R5, R6, R7, R9: (no value), biomimetic:RESISTOR0402-RES
- R3: value 1K -> (none); device OPL Eagle Library:R-4R -> biomimetic:RESISTOR0402-RES
Connections:
- net 3.3V: now also IC1P.V+; no longer C29.1, IC3P.V+, IC4P.V+
- net GND: now also IC1P.V-; no longer C29.2, IC3P.V-, IC4P.V-
- net MOTOR_A_BEMF: now also R3.2; no longer R3A.1
- net MOTOR_A_OUT1: now also R2.1; no longer R33B.2
- net MOTOR_A_OUT2: now also R4.1; no longer R33A.2
- net MOTOR_B_BEMF: now also R12.2; no longer R3B.1
- net MOTOR_B_OUT1: now also R5.1; no longer R33D.1
- net MOTOR_B_OUT2: now also R6.1; no longer R33C.1
- net MOTOR_C_BEMF: now also R13.2; no longer R3C.1
- net MOTOR_C_OUT1: now also R7.1; no longer R34A.1
- net MOTOR_C_OUT2: now also R9.1; no longer R34B.1
- net MOTOR_D_BEMF: now also R14.2; no longer R3D.1
- net MOTOR_D_OUT1: now also R10.1; no longer R34C.1
- net MOTOR_D_OUT2: now also R11.1; no longer R34D.1
- net N$22: now also IC1D.+IN, R5.2; no longer IC3B.+IN, R33D.2
- net N$23: now also IC1D.-IN, R6.2; no longer IC3B.-IN, R33C.2
- net N$24: now also IC1B.+IN, R7.2; no longer IC4A.+IN, R34A.2
- net N$25: now also IC1B.-IN, R9.2; no longer IC4A.-IN, R34B.2
- net N$26: now also IC1C.+IN, R10.2; no longer IC4B.+IN, R34C.2
- net N$27: now also IC1C.-IN, R11.2; no longer IC4B.-IN, R34D.2
- net N$30: now also IC1A.+IN, R2.2; no longer IC3A.+IN, R33B.1
- net N$31: now also IC1A.-IN, R4.2; no longer IC3A.-IN, R33A.1
- net N$34: now also IC1C.OUT, R14.1; no longer IC4B.OUT, R3D.2
- net N$35: now also IC1B.OUT, R13.1; no longer IC4A.OUT, R3C.2
- net N$36: now also IC1A.OUT, R3.1; no longer IC3A.OUT, R3A.2
- net N$37: now also IC1D.OUT, R12.1; no longer IC3B.OUT, R3B.2
